Commit message: Update robot.urdf.xacro

File: description/robot.urdf.xacro (robot description, xacro)
@@ -1,4 +1,5 @@
 <?xml version="1.0"?>
 <robot xmlns:xacro="http://www.ros.org/wiki/xacro"  name="robot">
-    <xacro:include filename="robot_core.xacro" />
+    <link name="base_link">
+    </link>
 </robot>

Commit message: 23/12

File: description/robot.urdf.xacro (robot description, xacro)
@@ -1,5 +1,6 @@
 <?xml version="1.0"?>
 <robot xmlns:xacro="http://www.ros.org/wiki/xacro"  name="robot">
-    <link name="base_link">
-    </link>
+    <xacro:include filename="inertial_macros.xacro" />
+    <xacro:include filename="robot_core.xacro" />
+    <xacro:include filename = "gazebo_control.xacro" />
 </robot>
