Commit message: 13/01

File: description/casterrobot_core.xacro (robot description, xacro)
@@ -19,4 +19,12 @@
     <link name="base_link">
     </link>
+    <!-- BASE_FOOTPRINT LINK -->
+<joint name="base_footprint_joint" type="fixed">
+ <parent link="base_link"/>
+ <child link="base_footprint"/>
+ <origin xyz="0 0 0" rpy="0 0 0"/>
+</joint>
+<link name="base_footprint">
+</link>
     <joint name="chassis_joint" type="fixed">
         <parent link="base_link"/>
